Commit message: Functional basic Gazebo Sim and Teleop_twist_keyboard for control

File: model/robot.xacro (robot description, xacro)
@@ -2,8 +2,6 @@
 <robot name="differential_drive_robot"
 xmlns:xacro="http://www.ros.org/wiki/xacro">
-<!--Geometry and constants-->
-<xacro:property name= "pi" value="3.14159"/>
 <!--Dimensions-->
-<xacro:property name="a" value="0.1"/>
+<xacro:property name="a" value="1"/>
 <xacro:property name="b" value="0.3"/>
 <xacro:property name="c" value="0.6"/>
@@ -70,5 +68,5 @@
     <visual>
         <geometry>
-          <box size="${a} ${b} ${c}"/>
+          <box size="${a} ${c} ${b}"/>
         </geometry>
         <origin rpy="0 0 0" xyz="0 0 ${s1}"/>
@@ -76,5 +74,5 @@
     <collision name="body_collision">
       <geometry>
-        <box size="${a} ${b} ${c}"/>
+        <box size="${a} ${c} ${b}"/>
       </geometry>
       <origin rpy="0 0 0" xyz="0 0 ${s1}"/>
@@ -93,5 +91,5 @@
   <link name="wheel1_link">
     <visual>
-      <origin rpy="1.57075 0 0" xyz="0 0 0"/>
+      <origin rpy="1.570795 0 0" xyz="0 0 0"/>
       <geometry>
         <cylinder length="${d}" radius="${r}"/>
@@ -99,5 +97,5 @@
     </visual>
     <collision>
-      <origin rpy="1.57075 0 0" xyz="0 0 0"/>
+      <origin rpy="1.570795 0 0" xyz="0 0 0"/>
       <geometry>
         <cylinder length="${d}" radius="${r}"/>
@@ -116,5 +114,5 @@
   <link name="wheel2_link">
     <visual>
-      <origin rpy="1.57075 0 0" xyz="0 0 0"/>
+      <origin rpy="1.570795 0 0" xyz="0 0 0"/>
       <geometry>
         <cylinder length="${d}" radius="${r}"/>
@@ -122,5 +120,5 @@
     </visual>
     <collision>
-      <origin rpy="1.57075 0 0" xyz="0 0 0"/>
+      <origin rpy="1.570795 0 0" xyz="0 0 0"/>
       <geometry>
         <cylinder length="${d}" radius="${r}"/>
